Commit message: Imported upstream version '0.5.5' of 'upstream'

File: schunk_description/urdf/lwa4p_extended/lwa4p_extended.gazebo.xacro (robot description, xacro)
@@ -2,43 +2,36 @@
 <robot xmlns:xacro="http://www.ros.org/wiki/xacro">
   <xacro:macro name="schunk_lwa4p_extended_gazebo" params="name">
-    <gazebo reference="${name}_0_link">
-      <material value="Schunk/LightGrey" />
-      <turnGravityOff>false</turnGravityOff>
-      <selfCollide>true</selfCollide>
+    <gazebo reference="${name}_base_link">
+      <gravity>true</gravity>
+      <self_collide>false</self_collide>
     </gazebo>
     <gazebo reference="${name}_1_link">
-      <material value="Schunk/LightGrey" />
-      <turnGravityOff>false</turnGravityOff>
-      <selfCollide>true</selfCollide>
+      <gravity>true</gravity>
+      <self_collide>false</self_collide>
     </gazebo>
     <gazebo reference="${name}_2_link">
-      <material value="Schunk/LightGrey" />
-      <turnGravityOff>false</turnGravityOff>
-      <selfCollide>true</selfCollide>
+      <gravity>true</gravity>
+      <self_collide>false</self_collide>
     </gazebo>
     <gazebo reference="${name}_3_link">
-      <material value="Schunk/LightGrey" />
-      <turnGravityOff>false</turnGravityOff>
-      <selfCollide>true</selfCollide>
+      <gravity>true</gravity>
+      <self_collide>false</self_collide>
     </gazebo>
     <gazebo reference="${name}_4_link">
-      <material value="Schunk/LightGrey" />
-      <turnGravityOff>false</turnGravityOff>
-      <selfCollide>true</selfCollide>
+      <gravity>true</gravity>
+      <self_collide>false</self_collide>
     </gazebo>
     <gazebo reference="${name}_5_link">
-      <material value="Schunk/LightGrey" />
-      <turnGravityOff>false</turnGravityOff>
-      <selfCollide>true</selfCollide>
+      <gravity>true</gravity>
+      <self_collide>false</self_collide>
     </gazebo>
     <gazebo reference="${name}_6_link">
-      <material value="Schunk/LightGrey" />
-      <turnGravityOff>false</turnGravityOff>
-      <selfCollide>true</selfCollide>
+      <gravity>true</gravity>
+      <self_collide>false</self_collide>
     </gazebo>
     <gazebo reference="${name}_7_link">
+      <gravity>true</gravity>
+      <self_collide>false</self_collide>
       <material value="Schunk/LightGrey" />
-      <turnGravityOff>false</turnGravityOff>
-      <selfCollide>true</selfCollide>
     </gazebo>
   </xacro:macro>

File: schunk_description/urdf/pg70/pg70.gazebo.xacro (robot description, xacro)
@@ -3,14 +3,17 @@
   <xacro:macro name="schunk_pg70_gazebo" params="name">
     <gazebo reference="${name}_palm_link">
+      <gravity>true</gravity>
+      <self_collide>false</self_collide>
       <material>Schunk/LightGrey</material>
-      <turnGravityOff>false</turnGravityOff>
     </gazebo>
-    <gazebo reference="${name}_finger_1_link">
+    <gazebo reference="${name}_finger_left_link">
+      <gravity>true</gravity>
+      <self_collide>false</self_collide>
       <material>Schunk/LightGrey</material>
-      <turnGravityOff>false</turnGravityOff>
     </gazebo>
-    <gazebo reference="${name}_finger_2_link">
+    <gazebo reference="${name}_finger_right_link">
+      <gravity>true</gravity>
+      <self_collide>false</self_collide>
       <material>Schunk/LightGrey</material>
-      <turnGravityOff>false</turnGravityOff>
     </gazebo>
   </xacro:macro>

File: schunk_description/urdf/pg70/pg70.transmission.xacro (robot description, xacro)
@@ -3,18 +3,20 @@
   <xacro:macro name="schunk_pg70_transmission" params="name">
     <!-- finger1 -->
-    <transmission name="${name}_finger_trans">
+    <transmission name="${name}_finger_left_trans">
       <type>transmission_interface/SimpleTransmission</type>
-      <joint name="${name}_finger_joint"/>
-      <actuator name="${name}_finger_motor">
+      <joint name="${name}_finger_left_joint">
         <hardwareInterface>EffortJointInterface</hardwareInterface>
+      </joint>
+      <actuator name="${name}_finger_left_motor">
         <mechanicalReduction>1</mechanicalReduction>
       </actuator>
     </transmission>
-    <!-- finger2 -->
-    <transmission name="${name}_finger_mimic_trans">
+    <!-- finger2 - mimic -->
+    <transmission name="${name}_finger_right_trans">
       <type>transmission_interface/SimpleTransmission</type>
-      <joint name="${name}_finger_mimic_joint"/>
-      <actuator name="${name}_finger_mimic_motor">
+      <joint name="${name}_finger_right_joint">
         <hardwareInterface>EffortJointInterface</hardwareInterface>
+      </joint>
+      <actuator name="${name}_finger_right_motor">
         <mechanicalReduction>1</mechanicalReduction>
       </actuator>

File: schunk_description/urdf/pg70/pg70.urdf.xacro (robot description, xacro)
@@ -1,98 +1,101 @@
 <?xml version="1.0"?>
 <robot xmlns:xacro="http://www.ros.org/wiki/xacro">
-  <xacro:include filename="$(find schunk_description)/urdf/materials.urdf.xacro" />
   <xacro:include filename="$(find schunk_description)/urdf/pg70/pg70.gazebo.xacro" />
   <xacro:include filename="$(find schunk_description)/urdf/pg70/pg70.transmission.xacro" />
-  <xacro:macro name="schunk_pg70" params="parent name *origin">
-    <!-- joint between arm_7_link and pg70_palm_link -->
+  <xacro:macro name="schunk_pg70" params="parent name *origin pg70_finger_left_ref pg70_finger_right_ref">
     <joint name="${name}_palm_joint" type="fixed" >
-      <insert_block name="origin" />
       <parent link="${parent}" />
       <child link="${name}_palm_link" />
+      <xacro:insert_block name="origin" />
     </joint>
     <link name="${name}_palm_link">
       <inertial>
         <origin xyz="0 0 0" rpy="0 0 0"/>
-        <mass value="1.0"/>
+        <mass value="1"/>
         <inertia ixx="0.01" ixy="0" ixz="0" iyy="0.01" iyz="0" izz="0.01" />
       </inertial>
       <visual>
-        <origin xyz="0 0 0.0465" rpy="0 0 0" />
         <geometry>
-          <box size="0.08 0.10 0.093"/>
+          <mesh filename="package://schunk_description/meshes/pg70/pg70.dae" />
         </geometry>
-        <material name="Schunk/LightGrey" />
+        <material name="blue">
+          <color rgba="0 0 1 1"/>
+        </material>
       </visual>
       <collision>
-        <origin xyz="0 0 0.0465" rpy="0 0 0" />
         <geometry>
-          <box size="0.075 0.095 0.085"/>
+          <mesh filename="package://schunk_description/meshes/pg70/pg70.dae" />
         </geometry>
+        <material name="blue">
+          <color rgba="0 0 1 1"/>
+        </material>
       </collision>
     </link>
-    <!-- finger1 -->
-    <!-- joint between pg70_palm_link and pg70_finger_1_link -->
-    <joint name="${name}_finger_joint" type="prismatic">
-      <origin xyz="0.0 0.03 0.093" rpy="0 0 0" />
-      <parent link="${name}_palm_link"/>
-      <child link="${name}_finger_1_link"/>
+    <joint name="${name}_finger_left_joint" type="prismatic" >
+      <parent link="${name}_palm_link" />
+      <child link="${name}_finger_left_link" />
+      <limit effort="100" lower="-0.001" upper="0.0345" velocity="2.0"/>
+      <calibration rising="${pg70_finger_left_ref}"/>
+      <origin xyz="0 0.0105 0.0789" rpy="0 0 0"/>
       <axis xyz="0 1 0" />
-      <dynamics damping="1" />
-      <limit effort="100" lower="0" upper="0.034" velocity="5"/>
     </joint>
-    <link name="${name}_finger_1_link">
+    <link name="${name}_finger_left_link">
       <inertial>
         <origin xyz="0 0 0" rpy="0 0 0"/>
-        <mass value="0.1"/>
+        <mass value="1"/>
         <inertia ixx="0.01" ixy="0" ixz="0" iyy="0.01" iyz="0" izz="0.01" />
       </inertial>
       <visual>
-        <origin xyz="0 0 0.03" rpy="0 0 0" />
         <geometry>
-          <box size="0.03 0.01 0.060"/>
+          <box size="0.03 0.01 0.01"/>
         </geometry>
-        <material name="Schunk/LightGrey" />
+        <material name="black">
+          <color rgba="0 0 0 1"/>
+        </material>
       </visual>
       <collision>
-        <origin xyz="0 0 0.03" rpy="0 0 0" />
         <geometry>
-          <box size="0.025 0.005 0.055"/>
+          <box size="0.03 0.01 0.01"/>
         </geometry>
+        <material name="black">
+          <color rgba="0 0 0 1"/>
+        </material>
       </collision>
     </link>
-    <!-- finger2 -->
-    <!-- joint between pg70_palm_link and pg70_finger_2_link -->
-    <joint name="${name}_finger_mimic_joint" type="prismatic">
-      <!--mimic joint="${name}_finger_joint" multiplier="1" offset="0"/-->
-      <origin xyz="0.0 -0.03 0.093" rpy="0 0 3.14" />
-      <parent link="${name}_palm_link"/>
-      <child link="${name}_finger_2_link"/>
-      <axis xyz="0 1 0" />
-      <dynamics damping="1" />
-      <limit effort="100" lower="0" upper="0.034" velocity="5"/>
+    <joint name="${name}_finger_right_joint" type="prismatic" >
+      <mimic joint="${name}_finger_left_joint" multiplier="1" offset="0"/>
+      <parent link="${name}_palm_link" />
+      <child link="${name}_finger_right_link" />
+      <limit effort="100" lower="-0.001" upper="0.0345" velocity="2.0"/>
+      <calibration rising="${pg70_finger_right_ref}"/>
+      <origin xyz="0 -0.0105 0.0789" rpy="-0 0 0"/>
+      <axis xyz="0 -1 0" />
     </joint>
-    <link name="${name}_finger_2_link">
+    <link name="${name}_finger_right_link">
       <inertial>
         <origin xyz="0 0 0" rpy="0 0 0"/>
-        <mass value="0.1"/>
+        <mass value="1"/>
         <inertia ixx="0.01" ixy="0" ixz="0" iyy="0.01" iyz="0" izz="0.01" />
       </inertial>
       <visual>
-        <origin xyz="0 0 0.03" rpy="0 0 0" />
         <geometry>
-          <box size="0.03 0.01 0.059"/>
+          <box size="0.03 0.01 0.01"/>
         </geometry>
-        <material name="Schunk/LightGrey" />
+        <material name="black">
+          <color rgba="0 0 0 1"/>
+        </material>
       </visual>
       <collision>
-        <origin xyz="0 0 0.03" rpy="0 0 0" />
         <geometry>
-          <box size="0.025 0.005 0.055"/>
+          <box size="0.03 0.01 0.01"/>
         </geometry>
+        <material name="black">
+          <color rgba="0 0 0 1"/>
+        </material>
       </collision>
     </link>
-    <!-- extensions -->
-    <xacro:schunk_pg70_gazebo name="${name}" />
-    <xacro:schunk_pg70_transmission name="${name}" />
+  <!-- extensions -->
+  <xacro:schunk_pg70_gazebo name="${name}" />
+  <xacro:schunk_pg70_transmission name="${name}" />
   </xacro:macro>
 </robot>
